File: WeatherStation.kicad_pcb (KiCad board)
At the start: 2 copper layers, 48 parts, among them IC1 TPS62901RPJR, J1 Conn_01x02, J2 Conn_01x02, SW1 SW_Push, U1 RP2040, U2 W25Q128JVSIQ, U3 RFM95W-868S2, U4 SHT30-DIS, U5 BMP280, U6 BH1750FVI-TR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

Commit message: PCB layout update
Parts:
- added J3: Conn_01x02, Connector_PinHeader_2.54mm:PinHeader_1x02_P2.54mm_Vertical, F.Cu at (85.1, 40.9)
- SW1: footprint Button_Switch_SMD:SW_Push_1P1T_NO_CK_KSC6xxJ -> Button_Switch_SMD:SW_SPST_TL3305A
- moved R10 46.3 mm to (62.0, 55.1), turned to 90 degrees
- moved C21 40.1 mm to (50.8, 49.8)
- moved R11 40.1 mm to (50.8, 48.0)
- moved R13 32.4 mm to (63.8, 55.1), turned to -90 degrees
- moved U6 31.3 mm to (55.1, 50.3), turned to 180 degrees
- moved C20 26.4 mm to (55.4, 48.0), turned to 0 degrees
- moved C13 23.9 mm to (55.4, 46.2), turned to 0 degrees
- moved U4 22.3 mm to (56.9, 55.4), turned to 0 degrees
- moved C19 21.9 mm to (87.6, 56.9), turned to 0 degrees
- moved C18 21.5 mm to (55.4, 44.5), turned to 0 degrees
- moved J1 20.5 mm to (77.0, 40.9), turned to -90 degrees
- moved R5 17.7 mm to (91.4, 45.8)
- moved R3 17.4 mm to (82.8, 46.2)
- moved SW1 17.2 mm to (83.6, 70.1), turned to 0 degrees
- moved IC1 17.0 mm to (86.6, 45.7)
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